File: Schematics/RevA/KiCad/Jot_RevA/Audio.kicad_sch (KiCad schematic)
At the start: 4 parts, among them Q2 AO3401A, U2 MMICT3902-00-012

Commit message: Audio sheet: Rec LED (R7 1k + D1 red) on MIC_VDD, U3 second mic DNP (left channel)
Co-Authored-By: Claude Opus 5.5 <noreply@anthropic.com>
Parts:
- added D1: Red, symbol Device:LED
- added R7: 1k, symbol Device:R
- added U3: MMICT3902-00-012, Sensor_Audio:Knowles_LGA-5_3.5x2.65mm, symbol Sensor_Audio:SPH0641LU4H-1
Connections:
- net GND: now also D1.1 (K), U3.3 (GND)
- net MIC_VDD: now also R7.1, U3.2 (SEL), U3.5 (VDD)
- net PDM_CLK: now also U3.4 (CLOCK)
- net PDM_DATA: now also U3.1 (DATA)
- new net: D1.2 (A), R7.2
Other:
- note added: "U3: second mic, not fitted on Rev A (DNP). SEL to MIC_VDD = left channel; U2 SEL to GND = right."

Commit message: Audio sheet: title block matches the other sheets
Co-Authored-By: Claude Opus 5.5 <noreply@anthropic.com>
Other:
- company: James Cronin -> James Donal Cronin
- title: Jot_RevA_Audio -> Jot Rev A: Audio
Changed lines of the file:
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@@
 	(paper "A4")
 	(title_block
-		(title "Jot_RevA_Audio")
+		(title "Jot Rev A: Audio")
 		(date "2026-10-03")
-		(rev "Rev A")
-		(company "James Cronin")
+		(rev "A")
+		(company "James Donal Cronin")
 	)
 	(symbol

Commit message: Audio sheet: mic uses a proper Jot:T3902 symbol
U2 and U3 used KiCad's Knowles SPH0641LU4H-1 symbol relabelled as the
T3902. They now use a Jot:T3902 library symbol with the TDK datasheet,
description and MPN (MMICT3902-00-012), and pin 2 named SELECT. The
Knowles LGA-5 footprint stays: pads, ground ring and port were checked
against the T3902 datasheet and match. Netlist (171 connections) and
ERC are unchanged. JOT-HW-001 open item 10 marked done.

Co-Authored-By: Claude Opus 5.5 <noreply@anthropic.com>
Parts:
- U2, U3: symbol Sensor_Audio:SPH0641LU4H-1 -> Jot:T3902
Changed lines of the file:
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@@
 	)
 	(symbol
-		(lib_id "Sensor_Audio:SPH0641LU4H-1")
+		(lib_id "Jot:T3902")
 		(at 139.7 101.6 0)
 		(unit 1)
@@
 			)
 		)
-		(property "Datasheet" "https://www.knowles.com/docs/default-source/model-downloads/sph0641lu4h-1-revb.pdf"
+		(property "Datasheet" "${KIPRJMOD}/../../Datasheets/Audio/T3902_TDK.pdf"
 			(at 139.7 101.6 0)
 			(show_name no)
@@
 			)
 		)
-		(property "Description" "Digital MEMS Microphone, LGA-5"
+		(property "Description" "TDK T3902 bottom-port PDM MEMS microphone, LGA-5 3.5x2.65 mm (MPN MMICT3902-00-012)"
 			(at 139.7 101.6 0)
 			(show_name no)
@@
 	)
 	(symbol
-		(lib_id "Sensor_Audio:SPH0641LU4H-1")
+		(lib_id "Jot:T3902")
 		(at 139.7 142.24 0)
 		(unit 1)
@@
 			)
 		)
-		(property "Datasheet" "https://www.knowles.com/docs/default-source/model-downloads/sph0641lu4h-1-revb.pdf"
+		(property "Datasheet" "${KIPRJMOD}/../../Datasheets/Audio/T3902_TDK.pdf"
 			(at 139.7 142.24 0)
 			(show_name no)
@@
 			)
 		)
-		(property "Description" "Digital MEMS Microphone, LGA-5"
+		(property "Description" "TDK T3902 bottom-port PDM MEMS microphone, LGA-5 3.5x2.65 mm (MPN MMICT3902-00-012)"
 			(at 139.7 142.24 0)
 			(show_name no)

Commit message: Footprints: all resistors (0402, R19 1206) and capacitors (0402, 10 uF 0603) assigned to match the BOM
Co-Authored-By: Claude Opus 5.5 <noreply@anthropic.com>
Parts:
- C11: footprint (none) -> Capacitor_SMD:C_0402_1005Metric
- R13, R7: footprint (none) -> Resistor_SMD:R_0402_1005Metric
Changed lines of the file:
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@@
 			)
 		)
-		(property "Footprint" ""
+		(property "Footprint" "Capacitor_SMD:C_0402_1005Metric"
 			(at 127 92.71 0)
 			(hide yes)
@@
 			)
 		)
-		(property "Footprint" ""
+		(property "Footprint" "Resistor_SMD:R_0402_1005Metric"
 			(at 116.84 92.71 0)
 			(hide yes)
@@
 			)
 		)
-		(property "Footprint" ""
+		(property "Footprint" "Resistor_SMD:R_0402_1005Metric"
 			(at 114.3 69.85 0)
 			(hide yes)

Commit message: Footprints: D1 LED 0603, D4 SOD-123, Y1 3215 crystal
Co-Authored-By: Claude Opus 5.5 <noreply@anthropic.com>
Parts:
- D1: footprint (none) -> LED_SMD:LED_0603_1608Metric
Changed lines of the file:
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@@
 			)
 		)
-		(property "Footprint" ""
+		(property "Footprint" "LED_SMD:LED_0603_1608Metric"
 			(at 116.84 100.33 0)
 			(hide yes)
