File: Schematics/RevA/KiCad/Jot_RevA/Storage.kicad_sch (KiCad schematic)
At the start: 0 parts

Commit message: Storage sheet: U2 W25Q01JV flash on +3V3 with 100 nF, QSPI labels
Co-Authored-By: Claude Opus 5.5 <noreply@anthropic.com>
Parts:
- added C10: 100nF, Package_SO:SOIC-8_3.9x4.9mm_P1.27mm, symbol Device:C
- added U2: W25Q01JVZEIQ, symbol Jot:W25Q01JVZEIQ
Connections:
- new net +3V3: C10.1, U2.8 (VCC)
- new net GND: C10.2, U2.4 (GND)
- new net QSPI_CSN: U2.1 (~{CS})
- new net QSPI_IO0: U2.5 (DI/IO0)
- new net QSPI_IO1: U2.2 (DO/IO1)
- new net QSPI_IO2: U2.3 (~{WP}/IO2)
- new net QSPI_IO3: U2.7 (~{HOLD}/IO3)
- new net QSPI_SCK: U2.6 (CLK)

Commit message: Storage sheet: flash is U4 (matches BOM)
Co-Authored-By: Claude Opus 5.5 <noreply@anthropic.com>
Parts:
- renumbered U2 to U4
Changed lines of the file:
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@@
 		(dnp no)
 		(fields_autoplaced yes)
-		(property "Reference" "U2"
+		(property "Reference" "U4"
 			(at 163.83 92.7099 0)
 			(show_name no)
@@
 			(project "Jot_RevA"
 				(path "/61747270-9f90-47b6-9c50-5ea1f41f259a/0b47c322-4767-4ab6-bf09-bf78d39931f5"
-					(reference "U2")
+					(reference "U4")
 					(unit 1)
 				)

Commit message: Sensors sheet: U7 LIS2DW12 wired (I2C, SA0 high = 0x19, INT1 to ACC_INT1); clear wrong footprints on C6, C7, C10, C12, C13, Y1
Co-Authored-By: Claude Opus 5.5 <noreply@anthropic.com>
Parts:
- C10: footprint Package_SO:SOIC-8_3.9x4.9mm_P1.27mm -> (none)
Changed lines of the file:
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@@
 			)
 		)
-		(property "Footprint" "Package_SO:SOIC-8_3.9x4.9mm_P1.27mm"
+		(property "Footprint" ""
 			(at 169.8752 90.17 0)
 			(hide yes)

Commit message: Schematic review fixes: R18 100k flash /CS pull-up, R19 10R buzzer series resistor, T3902 DATA pin tri-state (ERC clean); BOM quantities and pin list updated
Co-Authored-By: Claude Opus 5.5 <noreply@anthropic.com>
Parts:
- added R18: 100k, symbol Device:R
Connections:
- net +3V3: now also R18.1
- net QSPI_CSN: now also R18.2
Changed lines of the file:
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@@
+		)
+	)
+	(symbol
+		(lib_id "Device:R")
+		(at 140.97 80.01 0)
+		(unit 1)
+		(body_style 1)
+		(exclude_from_sim no)
+		(in_bom yes)
+		(on_board yes)
+		(in_pos_files yes)
+		(dnp no)
+		(property "Reference" "R18"
+			(at 138.43 78.74 0)
+			(show_name no)
+			(do_not_autoplace no)
+			(effects
+				(font
+					(size 1.27 1.27)
+				)
+				(justify right)
+			)
+		)
+		(property "Value" "100k"
+			(at 138.43 81.28 0)
+			(show_name no)
+			(do_not_autoplace no)
+			(effects
+				(font
+					(size 1.27 1.27)
+				)
+				(justify right)
+			)
+		)
+		(property "Footprint" ""
+			(at 140.97 80.01 0)
+			(show_name no)
+			(do_not_autoplace no)
+			(hide yes)
+			(effects
+				(font
+					(size 1.27 1.27)
+				)
+			)
+		)
+		(property "Datasheet" ""
+			(at 140.97 80.01 0)
+			(show_name no)
+			(do_not_autoplace no)
+			(hide yes)
+			(effects
+				(font
+					(size 1.27 1.27)
+				)
+			)
+		)
+		(property "Description" "Resistor"
+			(at 140.97 80.01 0)
+			(show_name no)
+			(do_not_autoplace no)
+			(hide yes)
+			(effects
+				(font
+					(size 1.27 1.27)
+				)
+			)
+		)
+		(pin "1"
+		)
+		(pin "2"
+		)
+		(instances
+			(project "Jot_RevA"
+				(path "/61747270-9f90-47b6-9c50-5ea1f41f259a/0b47c322-4767-4ab6-bf09-bf78d39931f5"
+					(reference "R18")
+					(unit 1)
+				)
+			)
+		)
+	)
+	(wire
+		(pts
+			(xy 140.97 83.82) (xy 140.97 86.36)
+		)
+		(stroke
+			(width 0)
+			(type default)
+		)
+	)
+	(junction
+		(at 140.97 86.36)
+		(diameter 0)
+		(color 0 0 0 0)
+	)
+	(symbol
+		(lib_id "power:+3V3")
+		(at 140.97 73.66 0)
+		(unit 1)
+		(body_style 1)
+		(exclude_from_sim no)
+		(in_bom yes)
+		(on_board yes)
+		(in_pos_files yes)
+		(dnp no)
+		(property "Reference" "#PWR070"
+			(at 140.97 77.47 0)
+			(show_name no)
+			(do_not_autoplace no)
+			(hide yes)
+			(effects
+				(font
+					(size 1.27 1.27)
+				)
+			)
+		)
+		(property "Value" "+3V3"
+			(at 140.97 70.104 0)
+			(show_name no)
+			(do_not_autoplace no)
+			(effects
+				(font
+					(size 1.27 1.27)
+				)
+			)
+		)
+		(property "Footprint" ""
+			(at 140.97 73.66 0)
+			(show_name no)
+			(do_not_autoplace no)
+			(hide yes)
+			(effects
+				(font
+					(size 1.27 1.27)
+				)
+			)
+		)
+		(property "Datasheet" ""
+			(at 140.97 73.66 0)
+			(show_name no)
+			(do_not_autoplace no)
+			(hide yes)
+			(effects
+				(font
+					(size 1.27 1.27)
+				)
+			)
+		)
+		(property "Description" "Power symbol creates a global label with name \"+3V3\""
+			(at 140.97 73.66 0)
+			(show_name no)
+			(do_not_autoplace no)
+			(hide yes)
+			(effects
+				(font
+					(size 1.27 1.27)
+				)
+			)
+		)
+		(pin "1"
+		)
+		(instances
+			(project "Jot_RevA"
+				(path "/61747270-9f90-47b6-9c50-5ea1f41f259a/0b47c322-4767-4ab6-bf09-bf78d39931f5"
+					(reference "#PWR070")
+					(unit 1)
+				)
+			)
+		)
+	)
+	(wire
+		(pts
+			(xy 140.97 73.66) (xy 140.97 76.2)
+		)
+		(stroke
+			(width 0)
+			(type default)
 		)
 	)

Commit message: Footprints: all resistors (0402, R19 1206) and capacitors (0402, 10 uF 0603) assigned to match the BOM
Co-Authored-By: Claude Opus 5.5 <noreply@anthropic.com>
Parts:
- C10: footprint (none) -> Capacitor_SMD:C_0402_1005Metric
- R18: footprint (none) -> Resistor_SMD:R_0402_1005Metric

Commit message: Footprints: U4 flash WSON-8 8x6 EP3.4x4.3 (Winbond 8.3), U6 fuel gauge DFN-8 2x2 EP0.9x1.3 (matches SnapEDA; confirm vs Maxim 21-0168)
Co-Authored-By: Claude Opus 5.5 <noreply@anthropic.com>
Parts:
- U4: footprint (none) -> Package_SON:WSON-8-1EP_8x6mm_P1.27mm_EP3.4x4.3mm
Changed lines of the file:
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@@
 			)
 		)
-		(property "Footprint" ""
+		(property "Footprint" "Package_SON:WSON-8-1EP_8x6mm_P1.27mm_EP3.4x4.3mm"
 			(at 152.4 93.98 0)
 			(hide yes)
