File: Schematics/RevA/KiCad/Jot_RevA/Storage.kicad_sch (KiCad schematic)
At the start: 3 parts, among them U4 W25Q01JVZEIQ

Commit message: Rev A schematic final: battery fuse, reverse protection, VBUS TVS, charge inhibit, 32 MB flash
Polyfuse F1 and reverse-polarity P-FET Q6 between J2 and +BATT; SMF5.0A TVS on
VBUS; firmware charge inhibit (Q7/Q8, R20/R21, CHG_INHIBIT on P1.11, charging on
by default); R19 10R 1 W 2512; I2C pull-ups 2.2k; 1k series resistor on BTN;
flash W25Q256JVEIQ (symbol renamed); TP1/TP2/TP6 and J2 labels; junction dots.
BOM, pin list and architecture draft 5 updated (section 4.14: protection summary
and known Rev A limitations). JLCPCB upload BOM added. ERC clean.
Parts:
- U4: value W25Q01JVZEIQ -> W25Q256JVEIQ; symbol Jot:W25Q01JVZEIQ -> Jot:W25Q256JVEIQ
Changed lines of the file:
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@@
 	)
 	(symbol
-		(lib_id "Jot:W25Q01JVZEIQ")
+		(lib_id "Jot:W25Q256JVEIQ")
 		(at 152.4 93.98 0)
 		(unit 1)
@@
 			)
 		)
-		(property "Value" "W25Q01JVZEIQ"
+		(property "Value" "W25Q256JVEIQ"
 			(at 147.32 102.87 0)
-			(hide yes)
 			(show_name no)
 			(do_not_autoplace no)
@@
 			)
 		)
-		(property "Datasheet" "${KIPRJMOD}/../../Datasheets/Storage/W25Q01JV_Winbond.pdf"
+		(property "Datasheet" "kicad-embed://storage.pdf"
 			(at 152.4 93.98 0)
 			(hide yes)
@@
 			)
 		)
-		(property "Description" "1 Gbit (128 MB) 3 V serial NOR flash, SPI / Dual / Quad SPI, WSON-8 8x6 mm (ZE)"
+		(property "Description" "256 Mbit (32 MB) 3 V serial NOR flash, SPI / Dual / Quad SPI, WSON-8 8x6 mm (E)"
 			(at 152.4 93.98 0)
 			(hide yes)
