File: Schematics/RevA/KiCad/Jot_RevA/sensors.kicad_sch (KiCad schematic)
At the start: 0 parts

Commit message: Sensors sheet: U7 LIS2DW12 wired (I2C, SA0 high = 0x19, INT1 to ACC_INT1); clear wrong footprints on C6, C7, C10, C12, C13, Y1
Co-Authored-By: Claude Opus 5.5 <noreply@anthropic.com>
Parts:
- added C12: 10uF, symbol Device:C
- added C13: 100nF, symbol Device:C
- added U7: LIS2DW12TR, LIS2DW12TR:LGA-12_L2.0-W2.0-P0.50-BL, symbol Jot:LIS2DW12TR
Connections:
- new net +3V3: C12.2, C13.2, U7.10 (VDDIO), U7.2 (CS), U7.3 (SDO/SA0), U7.9 (VDD)
- new net ACC_INT1: U7.12 (INT1)
- new net GND: C12.1, C13.1, U7.6 (GND), U7.7 (RES), U7.8 (GND)
- new net I2C_SCL: U7.1 (SCL/SPC)
- new net I2C_SDA: U7.4 (SDA/SDI/SDO)
- no-connect marks 0 -> 1

Commit message: Sensors sheet: I2C pull-ups R3 (SDA) and R4 (SCL), 4.7k to +3V3
Co-Authored-By: Claude Opus 5.5 <noreply@anthropic.com>
Parts:
- added R3, R4: 4.7k, symbol Device:R
Connections:
- net +3V3: now also R3.2, R4.1
- net I2C_SCL: now also R4.2
- net I2C_SDA: now also R3.1

Commit message: Sensors sheet: U8 DRV2605L on +BATT with REG/VDD 1 uF, I2C, HAPTIC_EN, IN/TRIG to GND, OUT+/OUT- to TP1/TP2 motor pads
Co-Authored-By: Claude Opus 5.5 <noreply@anthropic.com>
Parts:
- added C14, C15: 1uF, symbol Device:C
- added TP1, TP2: TestPoint, symbol Connector:TestPoint
- added U8: DRV2605LDGS, Package_SO:TSSOP-10_3x3mm_P0.5mm, symbol Driver:DRV2605LDGS
Connections:
- net GND: now also C14.2, C15.2, U8.4 (IN/TRIG), U8.8 (GND)
- net I2C_SCL: now also U8.2 (SCL)
- net I2C_SDA: now also U8.3 (SDA)
- new net: TP2.1, U8.9 (OUT-)
- new net: TP1.1, U8.7 (OUT+)
- new net: C14.1, U8.1 (REG)
- new net +BATT: C15.1, U8.10 (VDD)
- new net HAPTIC_EN: U8.5 (EN)
- no-connect marks 1 -> 2

Commit message: Footprints: all resistors (0402, R19 1206) and capacitors (0402, 10 uF 0603) assigned to match the BOM
Co-Authored-By: Claude Opus 5.5 <noreply@anthropic.com>
Parts:
- C12: footprint (none) -> Capacitor_SMD:C_0603_1608Metric
- C13, C14, C15: footprint (none) -> Capacitor_SMD:C_0402_1005Metric
- R3, R4: footprint (none) -> Resistor_SMD:R_0402_1005Metric
Changed lines of the file:
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@@
 			)
 		)
-		(property "Footprint" ""
+		(property "Footprint" "Resistor_SMD:R_0402_1005Metric"
 			(at 141.732 114.3 90)
 			(hide yes)
@@
 			)
 		)
-		(property "Footprint" ""
+		(property "Footprint" "Capacitor_SMD:C_0402_1005Metric"
 			(at 213.36 100.0252 0)
 			(hide yes)
@@
 			)
 		)
-		(property "Footprint" ""
+		(property "Footprint" "Resistor_SMD:R_0402_1005Metric"
 			(at 146.812 88.9 90)
 			(hide yes)
@@
 			)
 		)
-		(property "Footprint" ""
+		(property "Footprint" "Capacitor_SMD:C_0402_1005Metric"
 			(at 74.6252 115.57 0)
 			(hide yes)
@@
 			)
 		)
-		(property "Footprint" ""
+		(property "Footprint" "Capacitor_SMD:C_0402_1005Metric"
 			(at 63.1952 83.82 0)
 			(hide yes)
@@
 			)
 		)
-		(property "Footprint" ""
+		(property "Footprint" "Capacitor_SMD:C_0603_1608Metric"
 			(at 213.36 88.5952 0)
 			(hide yes)

Commit message: Footprints: debug pads TP3-TP9 1.0 mm, motor wire pads TP1/TP2 2.0 mm
Co-Authored-By: Claude Opus 5.5 <noreply@anthropic.com>
Parts:
- TP1, TP2: footprint (none) -> TestPoint:TestPoint_Pad_D2.0mm
Changed lines of the file:
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@@
 			)
 		)
-		(property "Footprint" ""
+		(property "Footprint" "TestPoint:TestPoint_Pad_D2.0mm"
 			(at 73.66 99.06 0)
 			(hide yes)
@@
 			)
 		)
-		(property "Footprint" ""
+		(property "Footprint" "TestPoint:TestPoint_Pad_D2.0mm"
 			(at 83.82 96.52 0)
 			(hide yes)

Commit message: Footprints: U7 LIS2DW12 -> Package_LGA:LGA-12_2x2mm_P0.5mm (checked vs ST Figure 18; ERC fully clean)
Co-Authored-By: Claude Opus 5.5 <noreply@anthropic.com>
Parts:
- U7: footprint LIS2DW12TR:LGA-12_L2.0-W2.0-P0.50-BL -> Package_LGA:LGA-12_2x2mm_P0.5mm
Changed lines of the file:
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@@
 			)
 		)
-		(property "Footprint" "LIS2DW12TR:LGA-12_L2.0-W2.0-P0.50-BL"
+		(property "Footprint" "Package_LGA:LGA-12_2x2mm_P0.5mm"
 			(at 166.37 118.11 0)
 			(hide yes)
