File: Schematics/RevA/KiCad/Jot_RevA/sensors.kicad_sch (KiCad schematic)
At the start: 10 parts, among them U7 LIS2DW12TR, U8 DRV2605LDGS

Commit message: Rev A schematic final: battery fuse, reverse protection, VBUS TVS, charge inhibit, 32 MB flash
Polyfuse F1 and reverse-polarity P-FET Q6 between J2 and +BATT; SMF5.0A TVS on
VBUS; firmware charge inhibit (Q7/Q8, R20/R21, CHG_INHIBIT on P1.11, charging on
by default); R19 10R 1 W 2512; I2C pull-ups 2.2k; 1k series resistor on BTN;
flash W25Q256JVEIQ (symbol renamed); TP1/TP2/TP6 and J2 labels; junction dots.
BOM, pin list and architecture draft 5 updated (section 4.14: protection summary
and known Rev A limitations). JLCPCB upload BOM added. ERC clean.
Parts:
- R3, R4: value 4.7k -> 2.2k
- TP1: value TestPoint -> MOTOR+ (LRA)
- TP2: value TestPoint -> MOTOR- (LRA)
Changed lines of the file:
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@@
 	(wire
 		(pts
-			(xy 143.51 118.11) (xy 143.51 121.92)
+			(xy 132.08 120.65) (xy 132.08 118.11)
 		)
 		(stroke
@@
 	(wire
 		(pts
+			(xy 143.51 120.65) (xy 143.51 118.11)
+		)
+		(stroke
+			(width 0)
+			(type default)
+		)
+	)
+	(wire
+		(pts
 			(xy 146.05 96.52) (xy 148.59 96.52)
 		)
@@
 		(pts
 			(xy 73.66 106.68) (xy 73.66 107.95)
+		)
+		(stroke
+			(width 0)
+			(type default)
+		)
+	)
+	(wire
+		(pts
+			(xy 132.08 120.65) (xy 143.51 120.65)
 		)
 		(stroke
@@
 			)
 		)
-		(property "Value" "4.7k"
+		(property "Value" "2.2k"
 			(at 146.05 115.5699 0)
 			(show_name no)
@@
 			)
 		)
-		(property "Value" "TestPoint"
+		(property "Value" "MOTOR- (LRA)"
 			(at 81.28 103.6319 0)
 			(show_name no)
@@
 			)
 		)
-		(property "Value" "4.7k"
+		(property "Value" "2.2k"
 			(at 151.13 90.1699 0)
 			(show_name no)
@@
 			)
 		)
-		(property "Value" "TestPoint"
+		(property "Value" "MOTOR+ (LRA)"
 			(at 81.28 94.4879 0)
 			(show_name no)
@@
 	(symbol
 		(lib_id "power:+3V3")
-		(at 143.51 121.92 180)
+		(at 132.08 118.11 0)
 		(unit 1)
 		(body_style 1)
@@
 		(fields_autoplaced yes)
 		(property "Reference" "#PWR044"
-			(at 143.51 118.11 0)
+			(at 132.08 121.92 0)
 			(hide yes)
 			(show_name no)
@@
 		)
 		(property "Value" "+3V3"
-			(at 143.51 127 0)
-			(show_name no)
-			(do_not_autoplace no)
-			(effects
-				(font
-					(size 1.27 1.27)
-				)
+			(at 134.62 116.8399 0)
+			(show_name no)
+			(do_not_autoplace no)
+			(effects
+				(font
+					(size 1.27 1.27)
+				)
+				(justify left)
 			)
 		)
 		(property "Footprint" ""
-			(at 143.51 121.92 0)
+			(at 132.08 118.11 0)
 			(hide yes)
 			(show_name no)
@@
 		)
 		(property "Datasheet" ""
-			(at 143.51 121.92 0)
+			(at 132.08 118.11 0)
 			(hide yes)
 			(show_name no)
@@
 		)
 		(property "Description" "Power symbol creates a global label with name \"+3V3\""
-			(at 143.51 121.92 0)
-			(hide yes)
-			(show_name no)
+			(at 132.08 118.11 0)
+			(hide yes)
+			(show_name no)
