File: Schematics/RevA/KiCad/Jot_RevA/Power.kicad_sch (KiCad schematic)
At the start: 16 parts, among them J1 USB-C, J2 Battery, U10 USBLC6-2SC6, U5 MCP73831T-2ACI/OT, U6 MAX17048, U9 TPS7A0233

Commit message: Footprints: all resistors (0402, R19 1206) and capacitors (0402, 10 uF 0603) assigned to match the BOM
Co-Authored-By: Claude Opus 5.5 <noreply@anthropic.com>
Parts:
- R1, R2, R6: footprint (none) -> Resistor_SMD:R_0402_1005Metric

Commit message: Footprints: U4 flash WSON-8 8x6 EP3.4x4.3 (Winbond 8.3), U6 fuel gauge DFN-8 2x2 EP0.9x1.3 (matches SnapEDA; confirm vs Maxim 21-0168)
Co-Authored-By: Claude Opus 5.5 <noreply@anthropic.com>
Parts:
- U6: footprint (none) -> Package_DFN_QFN:DFN-8-1EP_2x2mm_P0.5mm_EP0.9x1.3mm
Changed lines of the file:
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@@
 			)
 		)
-		(property "Footprint" ""
+		(property "Footprint" "Package_DFN_QFN:DFN-8-1EP_2x2mm_P0.5mm_EP0.9x1.3mm"
 			(at 205.74 135.89 0)
 			(hide yes)

Commit message: Footprints: D2 RGB LED (new project library Jot.pretty, built from TOGIALED pad layout), J1 HRO TYPE-C-31-M-12, J2 JST S2B-PH-SM4-TB; project fp-lib-table
Co-Authored-By: Claude Opus 5.5 <noreply@anthropic.com>
Parts:
- J1: footprint (none) -> Connector_USB:USB_C_Receptacle_HRO_TYPE-C-31-M-12
- J2: footprint (none) -> Connector_JST:JST_PH_S2B-PH-SM4-TB_1x02-1MP_P2.00mm_Horizontal
Changed lines of the file:
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@@
 			)
 		)
-		(property "Footprint" ""
+		(property "Footprint" "Connector_JST:JST_PH_S2B-PH-SM4-TB_1x02-1MP_P2.00mm_Horizontal"
 			(at 185.42 91.44 0)
 			(hide yes)
@@
 			)
 		)
-		(property "Footprint" ""
+		(property "Footprint" "Connector_USB:USB_C_Receptacle_HRO_TYPE-C-31-M-12"
 			(at 34.29 86.36 0)
 			(hide yes)
