File: Schematics/RevA/KiCad/Jot_RevA/Power.kicad_sch (KiCad schematic)
At the start: 16 parts, among them J1 USB-C, J2 Battery, U10 USBLC6-2SC6, U5 MCP73831T-2ACI/OT, U6 MAX17048, U9 TPS7A0233

Commit message: Rev A schematic final: battery fuse, reverse protection, VBUS TVS, charge inhibit, 32 MB flash
Polyfuse F1 and reverse-polarity P-FET Q6 between J2 and +BATT; SMF5.0A TVS on
VBUS; firmware charge inhibit (Q7/Q8, R20/R21, CHG_INHIBIT on P1.11, charging on
by default); R19 10R 1 W 2512; I2C pull-ups 2.2k; 1k series resistor on BTN;
flash W25Q256JVEIQ (symbol renamed); TP1/TP2/TP6 and J2 labels; junction dots.
BOM, pin list and architecture draft 5 updated (section 4.14: protection summary
and known Rev A limitations). JLCPCB upload BOM added. ERC clean.
Parts:
- added D5: SMF5.0A, Diode_SMD:D_SOD-123F, symbol Device:D_Zener
- added F1: SMD0805P050TF, Fuse:Fuse_0805_2012Metric, symbol Device:Polyfuse
- added Q6: AO3401A, Package_TO_SOT_SMD:SOT-23, symbol Transistor_FET:AO3401A
- added Q7, Q8: AO3400A, Package_TO_SOT_SMD:SOT-23, symbol Transistor_FET:AO3400A
- added R20, R21: 100k, Resistor_SMD:R_0402_1005Metric, symbol Device:R
Connections:
- net +BATT: now also Q6.2 (S); no longer J2.1 (Pin_1)
- net GND: now also D5.2 (A), Q6.1 (G), Q7.2 (S), Q8.2 (S), R21.2; no longer R6.2
- net VBUS: now also D5.1 (K), R20.2
- new net: Q7.1 (G), Q8.3 (D), R20.1
- new net: Q7.3 (D), R6.2
- new net BATT_FUSED: F1.2, Q6.3 (D)
- new net BATT_RAW: F1.1, J2.1 (Pin_1)
- new net CHG_INHIBIT: Q8.1 (G), R21.1
Other:
- note added: "1 = BATT+ (red), 2 = BATT− (black)"
- note added: "CHG_INHIBIT HIGH = charging off (Q8 on, Q7 off, PROG floats). LOW or MCU off = charging on (R20 holds Q7 on from VBUS)."
- moved on the sheet: C5, J2, U6

Commit message: Rev A layout complete: final routing and layout review fixes
- J2 is now two solder-wire holes (battery leads soldered): the JST-PH
  side-entry header is 5.5 mm tall and would not fit the 12.8 mm case.
  Removed from the JLCPCB BOM; BOM, architecture doc and case notes updated.
- LED drive pins re-assigned to match the transistor order:
  P1.08 red, P0.11 green, P0.12 blue. Pin list updated.
- No via drilled inside an SMD pad; no top-layer signal or via beside the
  crystal; 5 V branch removed from the power layer under the USB pair.
- R19 off the battery, C11 next to the mic, short ground vias at the
  module and decoupling capacitors, clean reset route.
- Silkscreen labels at 1.0 mm, battery + / - marked; zones refilled.
- DRC clean, board matches schematic, ERC clean.
- Case: 0.4 mm pocket over SW1, lip 0.8 mm.
- Architecture draft 7.
Parts:
- J2: value Battery -> Battery wires; footprint Connector_JST:JST_PH_S2B-PH-SM4-TB_1x02-1MP_P2.00mm_Horizontal -> Connector_Wire:SolderWire-0.15sqmm_1x02_P4mm_D0.5mm_OD1.5mm; now not fitted; now left out of the parts list
Changed lines of the file:
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@@
 		(comment 1 "JOT-HW-001: handheld push-to-talk voice capture")
+	)
+	(text "CHG_INHIBIT HIGH = charging off\n(Q8 on, Q7 off, PROG floats).\nLOW or MCU off = charging on\n(R20 holds Q7 on from VBUS)."
+		(exclude_from_sim no)
+		(at 149.86 139.7 0)
+		(effects
+			(font
+				(size 1.27 1.27)
+			)
+			(justify left bottom)
+		)
 	)
 	(text "1 = BATT+ (red), 2 = BATT− (black)"
@@
 				(justify left)
 			)
-		)
-	)
-	(text "CHG_INHIBIT HIGH = charging off\n(Q8 on, Q7 off, PROG floats).\nLOW or MCU off = charging on\n(R20 holds Q7 on from VBUS)."
-		(exclude_from_sim no)
-		(at 149.86 139.7 0)
-		(effects
-			(font
-				(size 1.27 1.27)
-			)
-			(justify left bottom)
 		)
 	)
@@
 		(body_style 1)
 		(exclude_from_sim no)
-		(in_bom yes)
+		(in_bom no)
 		(on_board yes)
-		(in_pos_files yes)
-		(dnp no)
+		(in_pos_files no)
+		(dnp yes)
 		(property "Reference" "J2"
 			(at 191.77 102.8699 0)
@@
 			)
 		)
-		(property "Value" "Battery"
+		(property "Value" "Battery wires"
 			(at 191.77 106.68 0)
 			(show_name no)
@@
 			)
 		)
-		(property "Footprint" "Connector_JST:JST_PH_S2B-PH-SM4-TB_1x02-1MP_P2.00mm_Horizontal"
+		(property "Footprint" "Connector_Wire:SolderWire-0.15sqmm_1x02_P4mm_D0.5mm_OD1.5mm"
 			(at 189.23 102.87 0)
 			(hide yes)
