File: Schematics/RevA/KiCad/Jot_RevA/UI.kicad_sch (KiCad schematic)
At the start: 16 parts, among them Q1 AO3400A, Q3 AO3400A, Q4 AO3400A, Q5 AO3400A, SW1 SW_Push

Commit message: Footprints: SW1 and BZ1 assigned (JLCPCB footprints); every symbol pin has a pad on its footprint, only AE1 (PCB coil) left for layout
Co-Authored-By: Claude Opus 5.5 <noreply@anthropic.com>
Parts:
- BZ1: footprint (none) -> Jot:BUZ-SMD_L5.0-W5.5-P4.60
- SW1: footprint (none) -> Jot:KEY-SMD_TX-1010-X-X
Changed lines of the file:
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@@
 			)
 		)
-		(property "Footprint" ""
+		(property "Footprint" "Jot:KEY-SMD_TX-1010-X-X"
 			(at 167.64 53.34 0)
 			(hide yes)
@@
 			)
 		)
-		(property "Footprint" ""
+		(property "Footprint" "Jot:BUZ-SMD_L5.0-W5.5-P4.60"
 			(at 99.695 104.14 90)
 			(hide yes)
