File: Schematics/RevA/KiCad/Jot_RevA/UI.kicad_sch (KiCad schematic)
At the start: 16 parts, among them Q1 AO3400A, Q3 AO3400A, Q4 AO3400A, Q5 AO3400A, SW1 SW_Push

Commit message: Rev A schematic final: battery fuse, reverse protection, VBUS TVS, charge inhibit, 32 MB flash
Polyfuse F1 and reverse-polarity P-FET Q6 between J2 and +BATT; SMF5.0A TVS on
VBUS; firmware charge inhibit (Q7/Q8, R20/R21, CHG_INHIBIT on P1.11, charging on
by default); R19 10R 1 W 2512; I2C pull-ups 2.2k; 1k series resistor on BTN;
flash W25Q256JVEIQ (symbol renamed); TP1/TP2/TP6 and J2 labels; junction dots.
BOM, pin list and architecture draft 5 updated (section 4.14: protection summary
and known Rev A limitations). JLCPCB upload BOM added. ERC clean.
Parts:
- added R5: 1k, Resistor_SMD:R_0402_1005Metric, symbol Device:R
- R19: footprint Resistor_SMD:R_1206_3216Metric -> Resistor_SMD:R_2512_6332Metric
Connections:
- net BTN: now also R5.2; no longer SW1.1
- new net: R5.1, SW1.1
Changed lines of the file:
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@@
+	(wire
+		(pts
+			(xy 149.86 48.26) (xy 162.56 48.26)
+		)
+		(stroke
+			(width 0)
+			(type default)
+		)
+	)
 	(wire
 		(pts
@@
 	(wire
 		(pts
+			(xy 134.62 48.26) (xy 142.24 48.26)
+		)
+		(stroke
+			(width 0)
+			(type default)
+		)
+	)
+	(wire
+		(pts
 			(xy 97.79 109.22) (xy 97.79 115.57)
 		)
@@
 		(pts
 			(xy 210.82 127) (xy 205.74 127)
-		)
-		(stroke
-			(width 0)
-			(type default)
-		)
-	)
-	(wire
-		(pts
-			(xy 146.05 48.26) (xy 162.56 48.26)
 		)
 		(stroke
@@
 	(global_label "BTN"
 		(shape output)
-		(at 146.05 48.26 180)
+		(at 134.62 48.26 180)
 		(fields_autoplaced yes)
 		(effects
@@
 		)
 		(property "Intersheetrefs" "${INTERSHEET_REFS}"
-			(at 139.4967 48.26 0)
+			(at 128.0667 48.26 0)
 			(hide yes)
 			(show_name no)
@@
 	)
 	(symbol
+		(lib_id "Device:R")
+		(at 146.05 48.26 270)
+		(unit 1)
+		(body_style 1)
+		(exclude_from_sim no)
+		(in_bom yes)
+		(on_board yes)
+		(in_pos_files yes)
+		(dnp no)
+		(fields_autoplaced yes)
+		(property "Reference" "R5"
+			(at 146.05 41.91 90)
+			(show_name no)
+			(do_not_autoplace no)
+			(effects
+				(font
+					(size 1.27 1.27)
+				)
+			)
+		)
+		(property "Value" "1k"
+			(at 146.05 44.45 90)
+			(show_name no)
+			(do_not_autoplace no)
+			(effects
+				(font
+					(size 1.27 1.27)
+				)
+			)
+		)
+		(property "Footprint" "Resistor_SMD:R_0402_1005Metric"
+			(at 146.05 46.482 90)
+			(hide yes)
+			(show_name no)
+			(do_not_autoplace no)
+			(effects
+				(font
+					(size 1.27 1.27)
+				)
+			)
+		)
+		(property "Datasheet" ""
+			(at 146.05 48.26 0)
+			(hide yes)
+			(show_name no)
+			(do_not_autoplace no)
+			(effects
+				(font
+					(size 1.27 1.27)
+				)
+			)
+		)
+		(property "Description" "Resistor"
+			(at 146.05 48.26 0)
+			(hide yes)
+			(show_name no)
+			(do_not_autoplace no)
+			(effects
+				(font
+					(size 1.27 1.27)
+				)
+			)
+		)
+		(pin "2"
+		)
+		(pin "1"
+		)
+		(instances
+			(project "Jot_RevA"
+				(path "/61747270-9f90-47b6-9c50-5ea1f41f259a/32fe5d00-0189-4157-8ea0-b1e59c92ae9f"
+					(reference "R5")
+					(unit 1)
+				)
+			)
+		)
+	)
+	(symbol
 		(lib_id "power:GND")
 		(at 162.56 68.58 0)
@@
 			)
 		)
-		(property "Footprint" "Resistor_SMD:R_1206_3216Metric"
+		(property "Footprint" "Resistor_SMD:R_2512_6332Metric"
 			(at 97.79 90.17 0)
 			(hide yes)
